Commit message: feat(g1): simulate abdominal basket deposit

File: dimos/robot/unitree/g1/g1.urdf (robot description, URDF)
Before this commit: robot g1_29dof_rev_1_0, 40 links, 39 joints
Links:
- added link basket_link, mass 0.05; collision box size=0.005 0.120 0.120; collision box size=0.210 0.005 0.120
Joints:
- added joint basket_joint: type fixed, parent pelvis, child basket_link, origin xyz=0.0614 0 -0.085 rpy=0 0 0

Commit message: feat(g1): use visual meshes for top-open basket deposit

File: dimos/robot/unitree/g1/g1.urdf (robot description, URDF)
Before this commit: robot g1_29dof_rev_1_0, 41 links, 40 joints
Links:
- link basket_link: geometry collision box size=0.005 0.120 0.120; collision box size=0.005 0.120 0.120
