Commit message: fix(g1-harvest): 重力補償URDFにGoPro質量(250g)を追加
g1_dex1_1_calibrated_550g.urdfのファイル名通りright_dex1_base_link+
finger×2の合計がちょうど550gで、GoProの質量が一切モデル化されていな
かった。model_no_kenshoの無指令(コマンドゼロ)実機テストで、これが
手先が常に下方向へドリフトする主因と実証できた(180g追加でドリフトが
ほぼ解消)。取付位置はDex1-1hand_UMIのdex1モード実測値を流用した概算。

Co-Authored-By: Claude Sonnet 5 <noreply@anthropic.com>

File: dimos/robot/unitree/g1/g1_dex1_1_calibrated_550g.urdf (robot description, URDF)
Before this commit: robot g1_29dof_mode_15, 42 links, 41 joints
Links:
- added link right_gopro_link, mass 0.25
Joints:
- added joint right_gopro_joint: type fixed, parent right_dex1_base_link, child right_gopro_link, origin xyz=0.02 0 0.06 rpy=0 0 0
